File: nggaguna.kicad_pcb (KiCad board)
At the start: 2 copper layers, 230.1 x 97.1 mm, 89 parts, among them U1 promicro

Commit message: revamp
Parts:
- added switch41: switch, footprints:200-minimal, F.Cu at (113.9, 107.3)
- added switch42: switch, footprints:200-minimal, F.Cu at (155.6, 107.3)
- moved diode37 29.1 mm to (131.0, 112.2)
- moved diode38 29.0 mm to (138.5, 112.1)
- moved switch40 19.6 mm to (146.4, 109.6)
- moved switch39 19.6 mm to (123.2, 109.6)
- moved diode33 11.4 mm to (118.9, 97.4), turned to 76 degrees
- moved diode34 10.9 mm to (150.9, 97.8), turned to 284 degrees
Routing:
- net ROW2: track 287.1 -> 365.0 mm
- net COLM0: track 35.1 -> 111.3 mm
- net ROW3: track 299.0 -> 252.3 mm
- net Net-(diode38-Pad2): track 6.24 -> 26.4 mm
- net Net-(diode37-Pad2): track 5.54 -> 21.6 mm
- net Net-(diode34-Pad2): track 19.6 -> 26.3 mm
- net Net-(diode33-Pad2): track 19.3 -> 24.6 mm
- net COL5: track 86.1 -> 87.1 mm
- net COL4: track 88.1 -> 88.7 mm
Other:
- board size 230.1 x 97.1 mm -> 230.1 x 100.1 mm
